Commit message: The Maze solving for my cobot pro 600 has been executed

File: install/mycobot_pro_600_moveit_config/share/mycobot_pro_600_moveit_config/config/mycobot_pro_600.ros2_control.xacro (robot description, xacro)
@@ -1 +1,54 @@
-/home/sanjay/Desktop/cobot600/src/mycobot_pro_600_moveit_config/config/mycobot_pro_600.ros2_control.xacro
+<?xml version="1.0"?>
+<robot xmlns:xacro="http://www.ros.org/wiki/xacro">
+    <xacro:macro name="mycobot_pro_600_ros2_control" params="name initial_positions_file">
+        <xacro:property name="initial_positions" value="${xacro.load_yaml(initial_positions_file)['initial_positions']}"/>
+        <ros2_control name="${name}" type="system">
+            <hardware>
+                <!-- By default, set up controllers for simulation. This won't work on real hardware -->
+                <plugin>mock_components/GenericSystem</plugin>
+            </hardware>
+            <joint name="joint2_to_joint1">
+                <command_interface name="position"/>
+                <state_interface name="position">
+                  <param name="initial_value">${initial_positions['joint2_to_joint1']}</param>
+                </state_interface>
+                <state_interface name="velocity"/>
+            </joint>
+            <joint name="joint3_to_joint2">
+                <command_interface name="position"/>
+                <state_interface name="position">
+                  <param name="initial_value">${initial_positions['joint3_to_joint2']}</param>
+                </state_interface>
+                <state_interface name="velocity"/>
+            </joint>
+            <joint name="joint4_to_joint3">
+                <command_interface name="position"/>
+                <state_interface name="position">
+                  <param name="initial_value">${initial_positions['joint4_to_joint3']}</param>
+                </state_interface>
+                <state_interface name="velocity"/>
+            </joint>
+            <joint name="joint5_to_joint4">
+                <command_interface name="position"/>
+                <state_interface name="position">
+                  <param name="initial_value">${initial_positions['joint5_to_joint4']}</param>
+                </state_interface>
+                <state_interface name="velocity"/>
+            </joint>
+            <joint name="joint6_to_joint5">
+                <command_interface name="position"/>
+                <state_interface name="position">
+                  <param name="initial_value">${initial_positions['joint6_to_joint5']}</param>
+                </state_interface>
+                <state_interface name="velocity"/>
+            </joint>
+            <joint name="joint6output_to_joint6">
+                <command_interface name="position"/>
+                <state_interface name="position">
+                  <param name="initial_value">${initial_positions['joint6output_to_joint6']}</param>
+                </state_interface>
+                <state_interface name="velocity"/>
+            </joint>
+        </ros2_control>
+    </xacro:macro>
+</robot>

File: install/mycobot_pro_600_moveit_config/share/mycobot_pro_600_moveit_config/config/mycobot_pro_600.urdf.xacro (robot description, xacro)
@@ -1 +1,9 @@
-/home/sanjay/Desktop/cobot600/src/mycobot_pro_600_moveit_config/config/mycobot_pro_600.urdf.xacro
+<?xml version="1.0"?>
+<robot xmlns:xacro="http://www.ros.org/wiki/xacro" name="mycobot_pro_600">
+    <xacro:arg name="initial_positions_file" default="initial_positions.yaml" />
+    <!-- Import mycobot_pro_600 urdf file -->
+    <xacro:include filename="$(find mycobot_pro_600)/urdf/mycobot_pro_600.urdf" />
+    <!-- Import control_xacro -->
+    <xacro:include filename="mycobot_pro_600.ros2_control.xacro" />
+    <xacro:mycobot_pro_600_ros2_control name="FakeSystem" initial_positions_file="$(arg initial_positions_file)"/>
+</robot>

File: src/mycobot_pro_600/urdf/mycobot_pro_600.urdf (robot description, URDF)
Before this commit: robot mycobot_pro_600, 8 links, 7 joints
Joints:
- joint vision_joint: origin xyz=-0.15 -0.25 0 rpy=0 0 3.14159 -> xyz=-0.25 0.0 0 rpy=0 0 3.14159
